Commit message: base_link -> base_footprint

File: husarion_ugv_description/urdf/lynx/body.urdf.xacro (robot description, xacro)
@@ -4,10 +4,4 @@
     name="body"
     params="wheel_radius imu_xyz imu_rpy">
-    <link name="base_footprint" />
-    <joint name="base_to_body_joint" type="fixed">
-      <origin xyz="0.0 0.0 ${wheel_radius}" rpy="0.0 0.0 0.0" />
-      <parent link="base_footprint" />
-      <child link="base_link" />
-    </joint>
     <link name="base_link">
       <visual>
@@ -33,4 +27,10 @@
       </inertial>
     </link>
+    <joint name="base_to_footprint_joint" type="fixed">
+      <origin xyz="0.0 0.0 -${wheel_radius}" rpy="0.0 0.0 0.0" />
+      <parent link="base_link" />
+      <child link="base_footprint" />
+    </joint>
+    <link name="base_footprint" />
     <joint name="base_to_user_compartment_joint" type="fixed">
       <origin xyz="0.0 0.0 0.00535" rpy="0.0 0.0 0.0" />
@@ -83,5 +83,5 @@
       </inertial>
     </link>
-    <joint name="body_to_imu_joint" type="fixed">
+    <joint name="base_to_imu_joint" type="fixed">
       <origin xyz="${imu_xyz}" rpy="${imu_rpy}" />
       <parent link="base_link" />
@@ -89,5 +89,5 @@
     </joint>
     <link name="imu_link" />
-    <joint name="body_to_cover_joint" type="fixed">
+    <joint name="base_to_cover_joint" type="fixed">
       <!-- TODO change to real value -->
       <origin xyz="0.0 0.0 0.2085" rpy="0.0 0.0 0.0" />

File: husarion_ugv_description/urdf/panther/body.urdf.xacro (robot description, xacro)
@@ -5,10 +5,4 @@
     name="body"
     params="wheel_radius imu_xyz imu_rpy">
-    <link name="base_footprint" />
-    <joint name="base_to_body_joint" type="fixed">
-      <origin xyz="0.0 0.0 ${wheel_radius}" rpy="0.0 0.0 0.0" />
-      <parent link="base_footprint" />
-      <child link="base_link" />
-    </joint>
     <link name="base_link">
       <visual>
@@ -33,5 +27,11 @@
       </inertial>
     </link>
-    <joint name="body_to_imu_joint" type="fixed">
+    <joint name="base_to_footprint_joint" type="fixed">
+      <origin xyz="0.0 0.0 -${wheel_radius}" rpy="0.0 0.0 0.0" />
+      <parent link="base_link" />
+      <child link="base_footprint" />
+    </joint>
+    <link name="base_footprint" />
+    <joint name="base_to_imu_joint" type="fixed">
       <origin xyz="${imu_xyz}" rpy="${imu_rpy}" />
       <parent link="base_link" />
@@ -39,5 +39,5 @@
     </joint>
     <link name="imu_link" />
-    <joint name="body_to_front_bumper_joint" type="fixed">
+    <joint name="base_to_front_bumper_joint" type="fixed">
       <origin xyz="0.362 0.0 0.0" rpy="0.0 0.0 0.0" />
       <parent link="base_link" />
@@ -51,5 +51,5 @@
     </joint>
     <link name="lights_channel_1_link" />
-    <joint name="body_to_rear_bumper_joint" type="fixed">
+    <joint name="base_to_rear_bumper_joint" type="fixed">
       <origin xyz="-0.362 0.0 0.0" rpy="0.0 0.0 ${pi}" />
       <parent link="base_link" />
@@ -63,5 +63,5 @@
     </joint>
     <link name="lights_channel_2_link" />
-    <joint name="body_to_cover_joint" type="fixed">
+    <joint name="base_to_cover_joint" type="fixed">
       <origin xyz="0.0 0.0 0.1715" rpy="0.0 0.0 0.0" />
       <parent link="base_link" />
