Commit message: Use base_link in configs

File: husarion_ugv_description/urdf/lynx/base.urdf.xacro (robot description, xacro)
@@ -11,9 +11,9 @@
       </visual>
       <collision>
-        <origin xyz="0.0 0.0 0.0745" rpy="0.0 0.0 0.0" />
+        <origin xyz="0.0 0.0 0.09" rpy="0.0 0.0 0.0" />
         <geometry>
           <!-- TODO change when models ready -->
           <!-- <mesh filename="package://husarion_ugv_descriptions/meshes/panther/body_collision.stl" /> -->
-          <box size="0.646 0.34 0.268" />
+          <box size="0.64 0.34 0.28" />
         </geometry>
       </collision>

File: husarion_ugv_description/urdf/lynx/lynx_macro.urdf.xacro (robot description, xacro)
@@ -14,5 +14,5 @@
     <xacro:property name="wheel_separation_x" value="0.35" />
     <!-- INCLUDE ROBOT PARTS DEFINITIONS -->
-    <xacro:include filename="$(find husarion_ugv_descriptions)/urdf/lynx/body.urdf.xacro" ns="body" />
+    <xacro:include filename="$(find husarion_ugv_descriptions)/urdf/lynx/base.urdf.xacro" ns="body" />
     <xacro:include filename="$(find husarion_ugv_descriptions)/urdf/common/gazebo.urdf.xacro" ns="gazebo" />
     <xacro:include filename="$(find husarion_ugv_descriptions)/urdf/common/wheel.urdf.xacro" ns="wheel" />

File: husarion_ugv_description/urdf/panther/panther_macro.urdf.xacro (robot description, xacro)
@@ -18,5 +18,5 @@
     <xacro:property name="wheel_separation_x" value="0.44" />
     <!-- INCLUDE ROBOT PARTS DEFINITIONS -->
-    <xacro:include filename="$(find husarion_ugv_descriptions)/urdf/panther/body.urdf.xacro" ns="body" />
+    <xacro:include filename="$(find husarion_ugv_descriptions)/urdf/panther/base.urdf.xacro" ns="body" />
     <xacro:include filename="$(find husarion_ugv_descriptions)/urdf/common/gazebo.urdf.xacro" ns="gazebo" />
     <xacro:include filename="$(find husarion_ugv_descriptions)/urdf/common/wheel.urdf.xacro" ns="wheel" />

Commit message: Add reling link

File: husarion_ugv_description/urdf/lynx/base.urdf.xacro (robot description, xacro)
@@ -96,4 +96,10 @@
     </joint>
     <link name="cover_link" />
+    <joint name="cover_to_reling_joint" type="fixed">
+      <origin xyz="0.0 0.0 0.0215" rpy="0.0 0.0 0.0" />
+      <parent link="cover_link" />
+      <child link="reling_link" />
+    </joint>
+    <link name="reling_link" />
   </xacro:macro>
 </robot>

File: husarion_ugv_description/urdf/panther/base.urdf.xacro (robot description, xacro)
@@ -64,9 +64,15 @@
     <link name="lights_channel_2_link" />
     <joint name="base_to_cover_joint" type="fixed">
-      <origin xyz="0.0 0.0 0.1715" rpy="0.0 0.0 0.0" />
+      <origin xyz="0.0 0.0 0.14" rpy="0.0 0.0 0.0" />
       <parent link="base_link" />
       <child link="cover_link" />
     </joint>
     <link name="cover_link" />
+    <joint name="cover_to_reling_joint" type="fixed">
+      <origin xyz="0.0 0.0 0.0215" rpy="0.0 0.0 0.0" />
+      <parent link="cover_link" />
+      <child link="reling_link" />
+    </joint>
+    <link name="reling_link" />
   </xacro:macro>
 </robot>

Commit message: fix

File: husarion_ugv_description/urdf/lynx/base.urdf.xacro (robot description, xacro)
@@ -97,5 +97,5 @@
     <link name="cover_link" />
     <joint name="cover_to_reling_joint" type="fixed">
-      <origin xyz="0.0 0.0 0.0215" rpy="0.0 0.0 0.0" />
+      <origin xyz="0.0 0.0 0.0315" rpy="0.0 0.0 0.0" />
       <parent link="cover_link" />
       <child link="reling_link" />

File: husarion_ugv_description/urdf/panther/base.urdf.xacro (robot description, xacro)
@@ -70,5 +70,5 @@
     <link name="cover_link" />
     <joint name="cover_to_reling_joint" type="fixed">
-      <origin xyz="0.0 0.0 0.0215" rpy="0.0 0.0 0.0" />
+      <origin xyz="0.0 0.0 0.0315" rpy="0.0 0.0 0.0" />
       <parent link="cover_link" />
       <child link="reling_link" />

Commit message: Typos

File: husarion_ugv_description/urdf/lynx/base.urdf.xacro (robot description, xacro)
@@ -96,10 +96,10 @@
     </joint>
     <link name="cover_link" />
-    <joint name="cover_to_reling_joint" type="fixed">
+    <joint name="cover_to_rails_joint" type="fixed">
       <origin xyz="0.0 0.0 0.0315" rpy="0.0 0.0 0.0" />
       <parent link="cover_link" />
-      <child link="reling_link" />
+      <child link="rails_link" />
     </joint>
-    <link name="reling_link" />
+    <link name="rails_link" />
   </xacro:macro>
 </robot>

File: husarion_ugv_description/urdf/panther/base.urdf.xacro (robot description, xacro)
@@ -69,10 +69,10 @@
     </joint>
     <link name="cover_link" />
-    <joint name="cover_to_reling_joint" type="fixed">
+    <joint name="cover_to_rails_joint" type="fixed">
       <origin xyz="0.0 0.0 0.0315" rpy="0.0 0.0 0.0" />
       <parent link="cover_link" />
-      <child link="reling_link" />
+      <child link="rails_link" />
     </joint>
-    <link name="reling_link" />
+    <link name="rails_link" />
   </xacro:macro>
 </robot>

Commit message: mount link

File: husarion_ugv_description/urdf/lynx/base.urdf.xacro (robot description, xacro)
@@ -96,10 +96,10 @@
     </joint>
     <link name="cover_link" />
-    <joint name="cover_to_rails_joint" type="fixed">
+    <joint name="cover_to_mount_joint" type="fixed">
       <origin xyz="0.0 0.0 0.0315" rpy="0.0 0.0 0.0" />
       <parent link="cover_link" />
-      <child link="rails_link" />
+      <child link="mount_link" />
     </joint>
-    <link name="rails_link" />
+    <link name="mount_link" />
   </xacro:macro>
 </robot>

File: husarion_ugv_description/urdf/panther/base.urdf.xacro (robot description, xacro)
@@ -69,10 +69,10 @@
     </joint>
     <link name="cover_link" />
-    <joint name="cover_to_rails_joint" type="fixed">
+    <joint name="cover_to_mount_joint" type="fixed">
       <origin xyz="0.0 0.0 0.0315" rpy="0.0 0.0 0.0" />
       <parent link="cover_link" />
-      <child link="rails_link" />
+      <child link="mount_link" />
     </joint>
-    <link name="rails_link" />
+    <link name="mount_link" />
   </xacro:macro>
 </robot>

Commit message: Update Lynx meshes

File: husarion_ugv_description/urdf/lynx/base.urdf.xacro (robot description, xacro)
@@ -11,14 +11,12 @@
       </visual>
       <collision>
-        <origin xyz="0.0 0.0 0.09" rpy="0.0 0.0 0.0" />
+        <origin xyz="0.0 0.0 0.0" rpy="0.0 0.0 0.0" />
         <geometry>
-          <!-- TODO change when models ready -->
-          <!-- <mesh filename="package://husarion_ugv_description/meshes/panther/body_collision.stl" /> -->
-          <box size="0.64 0.34 0.28" />
+          <mesh filename="package://husarion_ugv_description/meshes/lynx/base_collision.dae" />
         </geometry>
       </collision>
       <inertial>
         <origin xyz="0.0 0.0 0.0" rpy="0.0 0.0 0.0" />
-        <mass value="30.0" />
+        <mass value="30.656" />
         <!-- TODO calculate real interia -->
         <inertia ixx="0.46856"  ixy="0.0"     ixz="0.0"
@@ -33,54 +31,4 @@
     </joint>
     <link name="base_footprint" />
-    <joint name="base_to_user_compartment_joint" type="fixed">
-      <origin xyz="0.0 0.0 0.00535" rpy="0.0 0.0 0.0" />
-      <parent link="base_link" />
-      <child link="user_compartment_link" />
-    </joint>
-    <link name="user_compartment_link">
-      <visual>
-        <geometry>
-          <mesh filename="package://husarion_ugv_description/meshes/lynx/user_compartment.dae" />
-        </geometry>
-      </visual>
-      <!-- TODO change when models ready -->
-      <!-- <collision>
-        <geometry>
-          <mesh filename="package://husarion_ugv_description/meshes/panther/user_compartment_collision.stl" />
-        </geometry>
-      </collision> -->
-      <inertial>
-        <!-- TODO calculate real interia -->
-        <mass value="30.0" />
-        <inertia ixx="0.46856"  ixy="0.0"     ixz="0.0"
-                                iyy="1.22285" iyz="0.0"
-                                              izz="1.51185" />
-      </inertial>
-    </link>
-    <joint name="base_to_battery_joint" type="fixed">
-      <origin xyz="-0.2628 -0.07945 0.07265" rpy="0.0 0.0 0.0" />
-      <parent link="base_link" />
-      <child link="battery_link" />
-    </joint>
-    <link name="battery_link">
-      <visual>
-        <geometry>
-          <mesh filename="package://husarion_ugv_description/meshes/lynx/battery.dae" />
-        </geometry>
-      </visual>
-      <!-- TODO change when models ready -->
-      <!-- <collision>
-        <geometry>
-          <mesh filename="package://husarion_ugv_description/meshes/panther/battery_collision.stl" />
-        </geometry>
-      </collision> -->
-      <inertial>
-        <mass value="30.0" />
-        <!-- TODO calculate real interia -->
-        <inertia ixx="0.46856"  ixy="0.0"     ixz="0.0"
-                                iyy="1.22285" iyz="0.0"
-                                              izz="1.51185" />
-      </inertial>
-    </link>
     <joint name="base_to_imu_joint" type="fixed">
       <origin xyz="${imu_xyz}" rpy="${imu_rpy}" />
@@ -97,5 +45,5 @@
     <link name="cover_link" />
     <joint name="cover_to_mount_joint" type="fixed">
-      <origin xyz="0.0 0.0 0.0315" rpy="0.0 0.0 0.0" />
+      <origin xyz="0.0 0.0 0.02" rpy="0.0 0.0 0.0" />
       <parent link="cover_link" />
       <child link="mount_link" />

Commit message: fix dimensions

File: husarion_ugv_description/urdf/lynx/base.urdf.xacro (robot description, xacro)
@@ -19,8 +19,7 @@
         <origin xyz="0.0 0.0 0.0" rpy="0.0 0.0 0.0" />
         <mass value="30.656" />
-        <!-- TODO calculate real interia -->
-        <inertia ixx="0.46856"  ixy="0.0"     ixz="0.0"
-                                iyy="1.22285" iyz="0.0"
-                                              izz="1.51185" />
+        <inertia ixx="0.6572" ixy="0.0334"  ixz="0.1739"
+                              iyy="1.443"   iyz="0.0082"
+                                            izz="1.598" />
       </inertial>
     </link>
@@ -38,6 +37,5 @@
     <link name="imu_link" />
     <joint name="base_to_cover_joint" type="fixed">
-      <!-- TODO change to real value -->
-      <origin xyz="0.0 0.0 0.2085" rpy="0.0 0.0 0.0" />
+      <origin xyz="0.0 0.0 0.2098" rpy="0.0 0.0 0.0" />
       <parent link="base_link" />
       <child link="cover_link" />
@@ -45,5 +43,5 @@
     <link name="cover_link" />
     <joint name="cover_to_mount_joint" type="fixed">
-      <origin xyz="0.0 0.0 0.02" rpy="0.0 0.0 0.0" />
+      <origin xyz="0.0 0.0 0.0217" rpy="0.0 0.0 0.0" />
       <parent link="cover_link" />
       <child link="mount_link" />

Commit message: adjust COM

File: husarion_ugv_description/urdf/lynx/base.urdf.xacro (robot description, xacro)
@@ -17,5 +17,5 @@
       </collision>
       <inertial>
-        <origin xyz="0.0 0.0 0.0" rpy="0.0 0.0 0.0" />
+        <origin xyz="-0.052 0.001 0.038" rpy="0.0 0.0 0.0" />
         <mass value="30.656" />
         <inertia ixx="0.6572" ixy="0.0334"  ixz="0.1739"

File: husarion_ugv_description/urdf/panther/base.urdf.xacro (robot description, xacro)
@@ -19,6 +19,5 @@
       </collision>
       <inertial>
-        <!-- TODO Fix oringin -->
-        <origin xyz="0.0 0.0 0.0" rpy="0.0 0.0 0.0" />
+        <origin xyz="-0.008 0.01 0.029" rpy="0.0 0.0 0.0" />
         <mass value="43.0" />
         <inertia ixx="2.630036" ixy="-0.023480" ixz="0.052320"
