Commit message: husarion_ugv_description -> husarion_ugv_descriptions

File: husarion_ugv_description/urdf/lynx.urdf.xacro (robot description, xacro)
@@ -6,5 +6,5 @@
   <xacro:arg name="imu_rpy" default="0.0 0.0 -1.57" />
   <xacro:arg name="wheel_config_file"
-    default="$(find husarion_ugv_description)/config/WH05.yaml" />
+    default="$(find husarion_ugv_descriptions)/config/WH05.yaml" />
   <xacro:arg name="controller_config_file"
     default="$(find husarion_ugv_controller)/config/WH05_controller.yaml" />
@@ -12,5 +12,5 @@
     default="" />
   <xacro:arg name="namespace" default="" />
-  <xacro:include filename="$(find husarion_ugv_description)/urdf/lynx/lynx_macro.urdf.xacro" ns="husarion" />
+  <xacro:include filename="$(find husarion_ugv_descriptions)/urdf/lynx/lynx_macro.urdf.xacro" ns="husarion" />
   <xacro:husarion.lynx_robot
     use_sim="$(arg use_sim)"
@@ -21,5 +21,5 @@
     battery_config_file="$(arg battery_config_file)"
     namespace="$(arg namespace)" />
-  <xacro:arg name="components_config_path" default="$(find husarion_ugv_description)/config/components.yaml" />
+  <xacro:arg name="components_config_path" default="$(find husarion_ugv_descriptions)/config/components.yaml" />
   <xacro:property name="components_config_path_property" value="$(arg components_config_path)" />
   <xacro:unless value="${components_config_path_property == 'None'}">

File: husarion_ugv_description/urdf/lynx/body.urdf.xacro (robot description, xacro)
@@ -13,5 +13,5 @@
       <visual>
         <geometry>
-          <mesh filename="package://husarion_ugv_description/meshes/lynx/base.dae" />
+          <mesh filename="package://husarion_ugv_descriptions/meshes/lynx/base.dae" />
         </geometry>
       </visual>
@@ -20,5 +20,5 @@
         <geometry>
           <!-- TODO change when models ready -->
-          <!-- <mesh filename="package://husarion_ugv_description/meshes/panther/body_collision.stl" /> -->
+          <!-- <mesh filename="package://husarion_ugv_descriptions/meshes/panther/body_collision.stl" /> -->
           <box size="0.646 0.34 0.268" />
         </geometry>
@@ -41,5 +41,5 @@
       <visual>
         <geometry>
-          <mesh filename="package://husarion_ugv_description/meshes/lynx/user_compartment.dae" />
+          <mesh filename="package://husarion_ugv_descriptions/meshes/lynx/user_compartment.dae" />
         </geometry>
       </visual>
@@ -47,5 +47,5 @@
       <!-- <collision>
         <geometry>
-          <mesh filename="package://husarion_ugv_description/meshes/panther/user_compartment_collision.stl" />
+          <mesh filename="package://husarion_ugv_descriptions/meshes/panther/user_compartment_collision.stl" />
         </geometry>
       </collision> -->
@@ -66,5 +66,5 @@
       <visual>
         <geometry>
-          <mesh filename="package://husarion_ugv_description/meshes/lynx/battery.dae" />
+          <mesh filename="package://husarion_ugv_descriptions/meshes/lynx/battery.dae" />
         </geometry>
       </visual>
@@ -72,5 +72,5 @@
       <!-- <collision>
         <geometry>
-          <mesh filename="package://husarion_ugv_description/meshes/panther/battery_collision.stl" />
+          <mesh filename="package://husarion_ugv_descriptions/meshes/panther/battery_collision.stl" />
         </geometry>
       </collision> -->

File: husarion_ugv_description/urdf/lynx/lynx_macro.urdf.xacro (robot description, xacro)
@@ -14,7 +14,7 @@
     <xacro:property name="wheel_separation_x" value="0.35" />
     <!-- INCLUDE ROBOT PARTS DEFINITIONS -->
-    <xacro:include filename="$(find husarion_ugv_description)/urdf/lynx/body.urdf.xacro" ns="body" />
-    <xacro:include filename="$(find husarion_ugv_description)/urdf/common/gazebo.urdf.xacro" ns="gazebo" />
-    <xacro:include filename="$(find husarion_ugv_description)/urdf/common/wheel.urdf.xacro" ns="wheel" />
+    <xacro:include filename="$(find husarion_ugv_descriptions)/urdf/lynx/body.urdf.xacro" ns="body" />
+    <xacro:include filename="$(find husarion_ugv_descriptions)/urdf/common/gazebo.urdf.xacro" ns="gazebo" />
+    <xacro:include filename="$(find husarion_ugv_descriptions)/urdf/common/wheel.urdf.xacro" ns="wheel" />
     <!-- BODY DECLARATION -->
     <xacro:body.body

File: husarion_ugv_description/urdf/panther.urdf.xacro (robot description, xacro)
@@ -5,5 +5,5 @@
   <xacro:arg name="imu_rpy" default="0.0 0.0 -1.57" />
   <xacro:arg name="wheel_config_file"
-    default="$(find husarion_ugv_description)/config/WH01.yaml" />
+    default="$(find husarion_ugv_descriptions)/config/WH01.yaml" />
   <xacro:arg name="controller_config_file"
     default="$(find husarion_ugv_controller)/config/WH01_controller.yaml" />
@@ -11,5 +11,5 @@
     default="" />
   <xacro:arg name="namespace" default="" />
-  <xacro:include filename="$(find husarion_ugv_description)/urdf/panther/panther_macro.urdf.xacro" ns="husarion" />
+  <xacro:include filename="$(find husarion_ugv_descriptions)/urdf/panther/panther_macro.urdf.xacro" ns="husarion" />
   <xacro:husarion.panther_robot
     use_sim="$(arg use_sim)"
@@ -20,5 +20,5 @@
     battery_config_file="$(arg battery_config_file)"
     namespace="$(arg namespace)" />
-  <xacro:arg name="components_config_path" default="$(find husarion_ugv_description)/config/components.yaml" />
+  <xacro:arg name="components_config_path" default="$(find husarion_ugv_descriptions)/config/components.yaml" />
   <xacro:property name="components_config_path_property" value="$(arg components_config_path)" />
   <xacro:unless value="${components_config_path_property == 'None'}">

File: husarion_ugv_description/urdf/panther/body.urdf.xacro (robot description, xacro)
@@ -15,5 +15,5 @@
         <origin xyz="0.0 0.0 0.0" rpy="0.0 0.0 0.0" />
         <geometry>
-          <mesh filename="package://husarion_ugv_description/meshes/panther/base.dae" />
+          <mesh filename="package://husarion_ugv_descriptions/meshes/panther/base.dae" />
         </geometry>
       </visual>
@@ -21,5 +21,5 @@
         <origin xyz="0.0 0.0 0.0" rpy="0.0 0.0 0.0" />
         <geometry>
-          <mesh filename="package://husarion_ugv_description/meshes/panther/base_collision.stl" />
+          <mesh filename="package://husarion_ugv_descriptions/meshes/panther/base_collision.stl" />
         </geometry>
       </collision>

File: husarion_ugv_description/urdf/panther/panther_macro.urdf.xacro (robot description, xacro)
@@ -18,7 +18,7 @@
     <xacro:property name="wheel_separation_x" value="0.44" />
     <!-- INCLUDE ROBOT PARTS DEFINITIONS -->
-    <xacro:include filename="$(find husarion_ugv_description)/urdf/panther/body.urdf.xacro" ns="body" />
-    <xacro:include filename="$(find husarion_ugv_description)/urdf/common/gazebo.urdf.xacro" ns="gazebo" />
-    <xacro:include filename="$(find husarion_ugv_description)/urdf/common/wheel.urdf.xacro" ns="wheel" />
+    <xacro:include filename="$(find husarion_ugv_descriptions)/urdf/panther/body.urdf.xacro" ns="body" />
+    <xacro:include filename="$(find husarion_ugv_descriptions)/urdf/common/gazebo.urdf.xacro" ns="gazebo" />
+    <xacro:include filename="$(find husarion_ugv_descriptions)/urdf/common/wheel.urdf.xacro" ns="wheel" />
     <!-- BODY DECLARATION -->
     <xacro:body.body

Commit message: husarion_ugv_descriptions -> husarion_ugv_description

File: husarion_ugv_description/urdf/lynx.urdf.xacro (robot description, xacro)
@@ -6,5 +6,5 @@
   <xacro:arg name="imu_rpy" default="0.0 0.0 -1.57" />
   <xacro:arg name="wheel_config_file"
-    default="$(find husarion_ugv_descriptions)/config/WH05.yaml" />
+    default="$(find husarion_ugv_description)/config/WH05.yaml" />
   <xacro:arg name="controller_config_file"
     default="$(find husarion_ugv_controller)/config/WH05_controller.yaml" />
@@ -12,5 +12,5 @@
     default="" />
   <xacro:arg name="namespace" default="" />
-  <xacro:include filename="$(find husarion_ugv_descriptions)/urdf/lynx/lynx_macro.urdf.xacro" ns="husarion" />
+  <xacro:include filename="$(find husarion_ugv_description)/urdf/lynx/lynx_macro.urdf.xacro" ns="husarion" />
   <xacro:husarion.lynx_robot
     use_sim="$(arg use_sim)"
@@ -21,5 +21,5 @@
     battery_config_file="$(arg battery_config_file)"
     namespace="$(arg namespace)" />
-  <xacro:arg name="components_config_path" default="$(find husarion_ugv_descriptions)/config/components.yaml" />
+  <xacro:arg name="components_config_path" default="$(find husarion_ugv_description)/config/components.yaml" />
   <xacro:property name="components_config_path_property" value="$(arg components_config_path)" />
   <xacro:unless value="${components_config_path_property == 'None'}">

File: husarion_ugv_description/urdf/lynx/base.urdf.xacro (robot description, xacro)
@@ -7,5 +7,5 @@
       <visual>
         <geometry>
-          <mesh filename="package://husarion_ugv_descriptions/meshes/lynx/base.dae" />
+          <mesh filename="package://husarion_ugv_description/meshes/lynx/base.dae" />
         </geometry>
       </visual>
@@ -14,5 +14,5 @@
         <geometry>
           <!-- TODO change when models ready -->
-          <!-- <mesh filename="package://husarion_ugv_descriptions/meshes/panther/body_collision.stl" /> -->
+          <!-- <mesh filename="package://husarion_ugv_description/meshes/panther/body_collision.stl" /> -->
           <box size="0.64 0.34 0.28" />
         </geometry>
@@ -41,5 +41,5 @@
       <visual>
         <geometry>
-          <mesh filename="package://husarion_ugv_descriptions/meshes/lynx/user_compartment.dae" />
+          <mesh filename="package://husarion_ugv_description/meshes/lynx/user_compartment.dae" />
         </geometry>
       </visual>
@@ -47,5 +47,5 @@
       <!-- <collision>
         <geometry>
-          <mesh filename="package://husarion_ugv_descriptions/meshes/panther/user_compartment_collision.stl" />
+          <mesh filename="package://husarion_ugv_description/meshes/panther/user_compartment_collision.stl" />
         </geometry>
       </collision> -->
@@ -66,5 +66,5 @@
       <visual>
         <geometry>
-          <mesh filename="package://husarion_ugv_descriptions/meshes/lynx/battery.dae" />
+          <mesh filename="package://husarion_ugv_description/meshes/lynx/battery.dae" />
         </geometry>
       </visual>
@@ -72,5 +72,5 @@
       <!-- <collision>
         <geometry>
-          <mesh filename="package://husarion_ugv_descriptions/meshes/panther/battery_collision.stl" />
+          <mesh filename="package://husarion_ugv_description/meshes/panther/battery_collision.stl" />
         </geometry>
       </collision> -->

File: husarion_ugv_description/urdf/lynx/lynx_macro.urdf.xacro (robot description, xacro)
@@ -2,5 +2,5 @@
 <robot xmlns:xacro="http://wiki.ros.org/xacro">
   <xacro:macro
-    name="panther_robot"
+    name="lynx_robot"
     params="wheel_config_file
             controller_config_file
@@ -10,15 +10,11 @@
             imu_rpy:='0.0 0.0 -1.57'
             namespace:=''">
-    <xacro:if value="${use_sim}">
-      <xacro:property name="imu_xyz" value="-0.195 0.010 0.085" />
-      <xacro:property name="imu_rpy" value="0.000 -0.000 3.142" />
-    </xacro:if>
     <xacro:property name="ns" value='${namespace + "/" if namespace else ""}' />
     <xacro:property name="wheel_config" value="${xacro.load_yaml(wheel_config_file)}" />
-    <xacro:property name="wheel_separation_x" value="0.44" />
+    <xacro:property name="wheel_separation_x" value="0.35" />
     <!-- INCLUDE ROBOT PARTS DEFINITIONS -->
-    <xacro:include filename="$(find husarion_ugv_descriptions)/urdf/panther/base.urdf.xacro" ns="body" />
-    <xacro:include filename="$(find husarion_ugv_descriptions)/urdf/common/gazebo.urdf.xacro" ns="gazebo" />
-    <xacro:include filename="$(find husarion_ugv_descriptions)/urdf/common/wheel.urdf.xacro" ns="wheel" />
+    <xacro:include filename="$(find husarion_ugv_description)/urdf/lynx/base.urdf.xacro" ns="body" />
+    <xacro:include filename="$(find husarion_ugv_description)/urdf/common/gazebo.urdf.xacro" ns="gazebo" />
+    <xacro:include filename="$(find husarion_ugv_description)/urdf/common/wheel.urdf.xacro" ns="wheel" />
     <!-- BODY DECLARATION -->
     <xacro:body.body
@@ -43,5 +39,5 @@
       wheel_separation_x="${wheel_separation_x}"
       prefix="rr" />
-    <ros2_control name="${ns}panther_system" type="system">
+    <ros2_control name="${ns}lynx_system" type="system">
       <hardware>
         <xacro:if value="${use_sim}">
@@ -50,5 +46,5 @@
         </xacro:if>
         <xacro:unless value="${use_sim}">
-          <plugin>husarion_ugv_hardware_interfaces/PantherSystem</plugin>
+          <plugin>husarion_ugv_hardware_interfaces/LynxSystem</plugin>
           <param name="encoder_resolution">1600</param>
           <param name="gear_ratio">30.08</param>
@@ -60,6 +56,5 @@
           <param name="can_interface_name">robot_can</param>
           <param name="master_can_id">3</param>
-          <param name="front_driver_can_id">1</param>
-          <param name="rear_driver_can_id">2</param>
+          <param name="driver_can_id">1</param>
           <param name="sdo_operation_timeout_ms">100</param>
           <!-- Depends on frequency of the controller, more critical motors state are sent with
@@ -156,6 +151,7 @@
       <xacro:gazebo.controller config_file="${controller_config_file}" namespace="${namespace}" />
       <xacro:gazebo.imu reference_frame="imu_link" namespace="${namespace}" />
-      <xacro:gazebo.light reference_frame="lights_channel_1_link" name="lights_channel_1" topic="lights/channel_1_frame" namespace="${namespace}" />
-      <xacro:gazebo.light reference_frame="lights_channel_2_link" name="lights_channel_2" topic="lights/channel_2_frame" namespace="${namespace}" />
+      <!-- TODO Add lights visualization -->
+      <!-- <xacro:gazebo.light reference_frame="lights_channel_1_link" name="lights_channel_1" topic="lights/channel_1_frame" namespace="${namespace}" /> -->
+      <!-- <xacro:gazebo.light reference_frame="lights_channel_2_link" name="lights_channel_2" topic="lights/channel_2_frame" namespace="${namespace}" /> -->
     </xacro:if>
   </xacro:macro>

File: husarion_ugv_description/urdf/panther.urdf.xacro (robot description, xacro)
@@ -5,5 +5,5 @@
   <xacro:arg name="imu_rpy" default="0.0 0.0 -1.57" />
   <xacro:arg name="wheel_config_file"
-    default="$(find husarion_ugv_descriptions)/config/WH01.yaml" />
+    default="$(find husarion_ugv_description)/config/WH01.yaml" />
   <xacro:arg name="controller_config_file"
     default="$(find husarion_ugv_controller)/config/WH01_controller.yaml" />
@@ -11,5 +11,5 @@
     default="" />
   <xacro:arg name="namespace" default="" />
-  <xacro:include filename="$(find husarion_ugv_descriptions)/urdf/panther/panther_macro.urdf.xacro" ns="husarion" />
+  <xacro:include filename="$(find husarion_ugv_description)/urdf/panther/panther_macro.urdf.xacro" ns="husarion" />
   <xacro:husarion.panther_robot
     use_sim="$(arg use_sim)"
@@ -20,5 +20,5 @@
     battery_config_file="$(arg battery_config_file)"
     namespace="$(arg namespace)" />
-  <xacro:arg name="components_config_path" default="$(find husarion_ugv_descriptions)/config/components.yaml" />
+  <xacro:arg name="components_config_path" default="$(find husarion_ugv_description)/config/components.yaml" />
   <xacro:property name="components_config_path_property" value="$(arg components_config_path)" />
   <xacro:unless value="${components_config_path_property == 'None'}">

File: husarion_ugv_description/urdf/panther/base.urdf.xacro (robot description, xacro)
@@ -9,5 +9,5 @@
         <origin xyz="0.0 0.0 0.0" rpy="0.0 0.0 0.0" />
         <geometry>
-          <mesh filename="package://husarion_ugv_descriptions/meshes/panther/base.dae" />
+          <mesh filename="package://husarion_ugv_description/meshes/panther/base.dae" />
         </geometry>
       </visual>
@@ -15,5 +15,5 @@
         <origin xyz="0.0 0.0 0.0" rpy="0.0 0.0 0.0" />
         <geometry>
-          <mesh filename="package://husarion_ugv_descriptions/meshes/panther/base_collision.stl" />
+          <mesh filename="package://husarion_ugv_description/meshes/panther/base_collision.stl" />
         </geometry>
       </collision>

File: husarion_ugv_description/urdf/panther/panther_macro.urdf.xacro (robot description, xacro)
@@ -2,5 +2,5 @@
 <robot xmlns:xacro="http://wiki.ros.org/xacro">
   <xacro:macro
-    name="lynx_robot"
+    name="panther_robot"
     params="wheel_config_file
             controller_config_file
@@ -10,11 +10,15 @@
             imu_rpy:='0.0 0.0 -1.57'
             namespace:=''">
+    <xacro:if value="${use_sim}">
+      <xacro:property name="imu_xyz" value="-0.195 0.010 0.085" />
+      <xacro:property name="imu_rpy" value="0.000 -0.000 3.142" />
+    </xacro:if>
     <xacro:property name="ns" value='${namespace + "/" if namespace else ""}' />
     <xacro:property name="wheel_config" value="${xacro.load_yaml(wheel_config_file)}" />
-    <xacro:property name="wheel_separation_x" value="0.35" />
+    <xacro:property name="wheel_separation_x" value="0.44" />
     <!-- INCLUDE ROBOT PARTS DEFINITIONS -->
-    <xacro:include filename="$(find husarion_ugv_descriptions)/urdf/lynx/base.urdf.xacro" ns="body" />
-    <xacro:include filename="$(find husarion_ugv_descriptions)/urdf/common/gazebo.urdf.xacro" ns="gazebo" />
-    <xacro:include filename="$(find husarion_ugv_descriptions)/urdf/common/wheel.urdf.xacro" ns="wheel" />
+    <xacro:include filename="$(find husarion_ugv_description)/urdf/panther/base.urdf.xacro" ns="body" />
+    <xacro:include filename="$(find husarion_ugv_description)/urdf/common/gazebo.urdf.xacro" ns="gazebo" />
+    <xacro:include filename="$(find husarion_ugv_description)/urdf/common/wheel.urdf.xacro" ns="wheel" />
     <!-- BODY DECLARATION -->
     <xacro:body.body
@@ -39,5 +43,5 @@
       wheel_separation_x="${wheel_separation_x}"
       prefix="rr" />
-    <ros2_control name="${ns}lynx_system" type="system">
+    <ros2_control name="${ns}panther_system" type="system">
       <hardware>
         <xacro:if value="${use_sim}">
@@ -46,5 +50,5 @@
         </xacro:if>
         <xacro:unless value="${use_sim}">
-          <plugin>husarion_ugv_hardware_interfaces/LynxSystem</plugin>
+          <plugin>husarion_ugv_hardware_interfaces/PantherSystem</plugin>
           <param name="encoder_resolution">1600</param>
           <param name="gear_ratio">30.08</param>
@@ -56,5 +60,6 @@
           <param name="can_interface_name">robot_can</param>
           <param name="master_can_id">3</param>
-          <param name="driver_can_id">1</param>
+          <param name="front_driver_can_id">1</param>
+          <param name="rear_driver_can_id">2</param>
           <param name="sdo_operation_timeout_ms">100</param>
           <!-- Depends on frequency of the controller, more critical motors state are sent with
@@ -151,7 +156,6 @@
       <xacro:gazebo.controller config_file="${controller_config_file}" namespace="${namespace}" />
       <xacro:gazebo.imu reference_frame="imu_link" namespace="${namespace}" />
-      <!-- TODO Add lights visualization -->
-      <!-- <xacro:gazebo.light reference_frame="lights_channel_1_link" name="lights_channel_1" topic="lights/channel_1_frame" namespace="${namespace}" /> -->
-      <!-- <xacro:gazebo.light reference_frame="lights_channel_2_link" name="lights_channel_2" topic="lights/channel_2_frame" namespace="${namespace}" /> -->
+      <xacro:gazebo.light reference_frame="lights_channel_1_link" name="lights_channel_1" topic="lights/channel_1_frame" namespace="${namespace}" />
+      <xacro:gazebo.light reference_frame="lights_channel_2_link" name="lights_channel_2" topic="lights/channel_2_frame" namespace="${namespace}" />
     </xacro:if>
   </xacro:macro>
