Commit message: Add lynx mesh and use base_footprint

File: husarion_ugv_description/urdf/common/wheel.urdf.xacro (robot description, xacro)
@@ -29,5 +29,5 @@
     <joint name="${prefix}_wheel_joint" type="continuous">
       <origin xyz="${x} ${y} 0.0" rpy="0.0 0.0 0.0" />
-      <parent link="body_link" />
+      <parent link="base_link" />
       <child link="${prefix}_wheel_link" />
       <axis xyz="0.0 1.0 0.0" />
@@ -37,11 +37,7 @@
     <link name="${prefix}_wheel_link">
       <visual>
-        <origin xyz="0.0 0.0 0.0" rpy="-${pi/2} 0.0 0.0" />
+        <origin xyz="0.0 0.0 0.0" rpy="0.0 0.0 0.0" />
         <geometry>
-          <!-- TODO cheange when models ready -->
-          <!-- <mesh
-          filename="package://${wheel_config['mesh_package']}/${wheel_config['folder_path']}/${prefix}_wheel.dae"
-          /> -->
-          <cylinder radius="${wheel_config['wheel_radius']}" length="${wheel_config['wheel_width']}" />
+          <mesh filename="package://${wheel_config['mesh_package']}/${wheel_config['folder_path']}/${prefix}_wheel.dae" />
         </geometry>
       </visual>

File: husarion_ugv_description/urdf/lynx/body.urdf.xacro (robot description, xacro)
@@ -1,21 +1,17 @@
 <?xml version="1.0" encoding="utf-8"?>
 <robot xmlns:xacro="http://wiki.ros.org/xacro">
-  <!-- body defining macro -->
   <xacro:macro
     name="body"
     params="wheel_radius imu_xyz imu_rpy">
-    <link name="base_link" />
+    <link name="base_footprint" />
     <joint name="base_to_body_joint" type="fixed">
       <origin xyz="0.0 0.0 ${wheel_radius}" rpy="0.0 0.0 0.0" />
-      <parent link="base_link" />
-      <child link="body_link" />
+      <parent link="base_footprint" />
+      <child link="base_link" />
     </joint>
-    <link name="body_link">
+    <link name="base_link">
       <visual>
-        <origin xyz="0.0 0.0 0.0745" rpy="0.0 0.0 0.0" />
         <geometry>
-          <!-- TODO cheange when models ready -->
-          <!-- <mesh filename="package://husarion_ugv_description/meshes/panther/body.dae" /> -->
-          <box size="0.646 0.34 0.268" />
+          <mesh filename="package://husarion_ugv_description/meshes/lynx/base.dae" />
         </geometry>
       </visual>
@@ -23,5 +19,5 @@
         <origin xyz="0.0 0.0 0.0745" rpy="0.0 0.0 0.0" />
         <geometry>
-          <!-- TODO cheange when models ready -->
+          <!-- TODO change when models ready -->
           <!-- <mesh filename="package://husarion_ugv_description/meshes/panther/body_collision.stl" /> -->
           <box size="0.646 0.34 0.268" />
@@ -37,14 +33,64 @@
       </inertial>
     </link>
+    <joint name="base_to_user_compartment_joint" type="fixed">
+      <origin xyz="0.0 0.0 0.00535" rpy="0.0 0.0 0.0" />
+      <parent link="base_link" />
+      <child link="user_compartment_link" />
+    </joint>
+    <link name="user_compartment_link">
+      <visual>
+        <geometry>
+          <mesh filename="package://husarion_ugv_description/meshes/lynx/user_compartment.dae" />
+        </geometry>
+      </visual>
+      <!-- TODO change when models ready -->
+      <!-- <collision>
+        <geometry>
+          <mesh filename="package://husarion_ugv_description/meshes/panther/user_compartment_collision.stl" />
+        </geometry>
+      </collision> -->
+      <inertial>
+        <!-- TODO calculate real interia -->
+        <mass value="30.0" />
+        <inertia ixx="0.46856"  ixy="0.0"     ixz="0.0"
+                                iyy="1.22285" iyz="0.0"
+                                              izz="1.51185" />
+      </inertial>
+    </link>
+    <joint name="base_to_battery_joint" type="fixed">
+      <origin xyz="-0.2628 -0.07945 0.07265" rpy="0.0 0.0 0.0" />
+      <parent link="base_link" />
+      <child link="battery_link" />
+    </joint>
+    <link name="battery_link">
+      <visual>
+        <geometry>
+          <mesh filename="package://husarion_ugv_description/meshes/lynx/battery.dae" />
+        </geometry>
+      </visual>
+      <!-- TODO change when models ready -->
+      <!-- <collision>
+        <geometry>
+          <mesh filename="package://husarion_ugv_description/meshes/panther/battery_collision.stl" />
+        </geometry>
+      </collision> -->
+      <inertial>
+        <mass value="30.0" />
+        <!-- TODO calculate real interia -->
+        <inertia ixx="0.46856"  ixy="0.0"     ixz="0.0"
+                                iyy="1.22285" iyz="0.0"
+                                              izz="1.51185" />
+      </inertial>
+    </link>
     <joint name="body_to_imu_joint" type="fixed">
       <origin xyz="${imu_xyz}" rpy="${imu_rpy}" />
-      <parent link="body_link" />
+      <parent link="base_link" />
       <child link="imu_link" />
     </joint>
     <link name="imu_link" />
     <joint name="body_to_cover_joint" type="fixed">
-      <!-- TODO cheange to real value -->
+      <!-- TODO change to real value -->
       <origin xyz="0.0 0.0 0.2085" rpy="0.0 0.0 0.0" />
-      <parent link="body_link" />
+      <parent link="base_link" />
       <child link="cover_link" />
     </joint>

File: husarion_ugv_description/urdf/lynx/lynx_macro.urdf.xacro (robot description, xacro)
@@ -22,5 +22,5 @@
     <xacro:include filename="$(find husarion_ugv_description)/urdf/lynx/body.urdf.xacro" ns="body" />
     <xacro:include filename="$(find husarion_ugv_description)/urdf/common/gazebo.urdf.xacro" ns="gazebo" />
-    <xacro:include filename="$(find husarion_ugv_description)/urdf/lynx/wheel.urdf.xacro" ns="wheel" />
+    <xacro:include filename="$(find husarion_ugv_description)/urdf/common/wheel.urdf.xacro" ns="wheel" />
     <!-- BODY DECLARATION -->
     <xacro:body.body

File: husarion_ugv_description/urdf/panther/body.urdf.xacro (robot description, xacro)
@@ -5,15 +5,15 @@
     name="body"
     params="wheel_radius imu_xyz imu_rpy">
-    <link name="base_link" />
+    <link name="base_footprint" />
     <joint name="base_to_body_joint" type="fixed">
       <origin xyz="0.0 0.0 ${wheel_radius}" rpy="0.0 0.0 0.0" />
-      <parent link="base_link" />
-      <child link="body_link" />
+      <parent link="base_footprint" />
+      <child link="base_link" />
     </joint>
-    <link name="body_link">
+    <link name="base_link">
       <visual>
         <origin xyz="0.0 0.0 0.0" rpy="0.0 0.0 0.0" />
         <geometry>
-          <mesh filename="package://husarion_ugv_description/meshes/panther/body.dae" />
+          <mesh filename="package://husarion_ugv_description/meshes/panther/base.dae" />
         </geometry>
       </visual>
@@ -21,8 +21,9 @@
         <origin xyz="0.0 0.0 0.0" rpy="0.0 0.0 0.0" />
         <geometry>
-          <mesh filename="package://husarion_ugv_description/meshes/panther/body_collision.stl" />
+          <mesh filename="package://husarion_ugv_description/meshes/panther/base_collision.stl" />
         </geometry>
       </collision>
       <inertial>
+        <!-- TODO: Fix oringin -->
         <origin xyz="0.0 0.0 0.0" rpy="0.0 0.0 0.0" />
         <mass value="43.0" />
@@ -34,5 +35,5 @@
     <joint name="body_to_imu_joint" type="fixed">
       <origin xyz="${imu_xyz}" rpy="${imu_rpy}" />
-      <parent link="body_link" />
+      <parent link="base_link" />
       <child link="imu_link" />
     </joint>
@@ -40,5 +41,5 @@
     <joint name="body_to_front_bumper_joint" type="fixed">
       <origin xyz="0.362 0.0 0.0" rpy="0.0 0.0 0.0" />
-      <parent link="body_link" />
+      <parent link="base_link" />
       <child link="front_bumper_link" />
     </joint>
@@ -52,5 +53,5 @@
     <joint name="body_to_rear_bumper_joint" type="fixed">
       <origin xyz="-0.362 0.0 0.0" rpy="0.0 0.0 ${pi}" />
-      <parent link="body_link" />
+      <parent link="base_link" />
       <child link="rear_bumper_link" />
     </joint>
@@ -64,5 +65,5 @@
     <joint name="body_to_cover_joint" type="fixed">
       <origin xyz="0.0 0.0 0.1715" rpy="0.0 0.0 0.0" />
-      <parent link="body_link" />
+      <parent link="base_link" />
       <child link="cover_link" />
     </joint>

File: husarion_ugv_description/urdf/panther/panther_macro.urdf.xacro (robot description, xacro)
@@ -20,5 +20,5 @@
     <xacro:include filename="$(find husarion_ugv_description)/urdf/panther/body.urdf.xacro" ns="body" />
     <xacro:include filename="$(find husarion_ugv_description)/urdf/common/gazebo.urdf.xacro" ns="gazebo" />
-    <xacro:include filename="$(find husarion_ugv_description)/urdf/panther/wheel.urdf.xacro" ns="wheel" />
+    <xacro:include filename="$(find husarion_ugv_description)/urdf/common/wheel.urdf.xacro" ns="wheel" />
     <!-- BODY DECLARATION -->
     <xacro:body.body

Commit message: use wheel mount point instead of wheel separation

File: husarion_ugv_description/urdf/common/wheel.urdf.xacro (robot description, xacro)
@@ -2,32 +2,43 @@
 <robot xmlns:xacro="http://wiki.ros.org/xacro">
   <!-- wheel defining macro -->
-  <xacro:macro name="wheel" params="wheel_config wheel_separation_x prefix">
+  <xacro:macro name="wheel"
+    params="wheel_config prefix wheel_mount_point_x wheel_mount_point_y">
     <xacro:if value="${prefix == 'fl'}">
-      <xacro:property name="x" value="${wheel_separation_x/2.0}" />
-      <xacro:property name="y" value="${wheel_config['wheel_separation']/2.0}" />
+      <xacro:property name="x" value="${wheel_mount_point_x}" />
+      <xacro:property name="y" value="${wheel_mount_point_y}" />
+      <xacro:property name="mount_point_offset" value="${wheel_config['mount_point_offset']}" />
       <xacro:property name="inertia_y_offset" value="${wheel_config['inertia_y_offset']}" />
       <xacro:property name="fdir" value="1 -1 0" />
     </xacro:if>
     <xacro:if value="${prefix == 'fr'}">
-      <xacro:property name="x" value="${wheel_separation_x/2.0}" />
-      <xacro:property name="y" value="-${wheel_config['wheel_separation']/2.0}" />
+      <xacro:property name="x" value="${wheel_mount_point_x}" />
+      <xacro:property name="y" value="-${wheel_mount_point_y}" />
+      <xacro:property name="mount_point_offset" value="-${wheel_config['mount_point_offset']}" />
       <xacro:property name="inertia_y_offset" value="${-wheel_config['inertia_y_offset']}" />
       <xacro:property name="fdir" value="1 1 0" />
     </xacro:if>
     <xacro:if value="${prefix == 'rl'}">
-      <xacro:property name="x" value="-${wheel_separation_x/2.0}" />
-      <xacro:property name="y" value="${wheel_config['wheel_separation']/2.0}" />
+      <xacro:property name="x" value="-${wheel_mount_point_x}" />
+      <xacro:property name="y" value="${wheel_mount_point_y}" />
+      <xacro:property name="mount_point_offset" value="${wheel_config['mount_point_offset']}" />
       <xacro:property name="inertia_y_offset" value="${wheel_config['inertia_y_offset']}" />
       <xacro:property name="fdir" value="1 1 0" />
     </xacro:if>
     <xacro:if value="${prefix == 'rr'}">
-      <xacro:property name="x" value="-${wheel_separation_x/2.0}" />
-      <xacro:property name="y" value="-${wheel_config['wheel_separation']/2.0}" />
+      <xacro:property name="x" value="-${wheel_mount_point_x}" />
+      <xacro:property name="y" value="-${wheel_mount_point_y}" />
+      <xacro:property name="mount_point_offset" value="-${wheel_config['mount_point_offset']}" />
       <xacro:property name="inertia_y_offset" value="${-wheel_config['inertia_y_offset']}" />
       <xacro:property name="fdir" value="1 -1 0" />
     </xacro:if>
-    <joint name="${prefix}_wheel_joint" type="continuous">
+    <joint name="base_to_${prefix}_wheel_base_joint" type="fixed">
       <origin xyz="${x} ${y} 0.0" rpy="0.0 0.0 0.0" />
       <parent link="base_link" />
+      <child link="${prefix}_wheel_base_link" />
+    </joint>
+    <link name="${prefix}_wheel_base_link" />
+    <joint name="${prefix}_wheel_joint" type="continuous">
+      <origin xyz="0.0 ${mount_point_offset} 0.0" rpy="0.0 0.0 0.0" />
+      <parent link="${prefix}_wheel_base_link" />
       <child link="${prefix}_wheel_link" />
       <axis xyz="0.0 1.0 0.0" />

File: husarion_ugv_description/urdf/lynx/lynx_macro.urdf.xacro (robot description, xacro)
@@ -12,5 +12,6 @@
     <xacro:property name="ns" value='${namespace + "/" if namespace else ""}' />
     <xacro:property name="wheel_config" value="${xacro.load_yaml(wheel_config_file)}" />
-    <xacro:property name="wheel_separation_x" value="0.35" />
+    <xacro:property name="wheelbase" value="0.35" />
+    <xacro:property name="wheel_mount_point_y" value="0.1675" />
     <!-- INCLUDE ROBOT PARTS DEFINITIONS -->
     <xacro:include filename="$(find husarion_ugv_description)/urdf/lynx/base.urdf.xacro" ns="body" />
@@ -25,17 +26,21 @@
     <xacro:wheel.wheel
       wheel_config="${wheel_config}"
-      wheel_separation_x="${wheel_separation_x}"
+      wheel_mount_point_x="${wheelbase/2.0}"
+      wheel_mount_point_y="${wheel_mount_point_y}"
       prefix="fl" />
     <xacro:wheel.wheel
       wheel_config="${wheel_config}"
-      wheel_separation_x="${wheel_separation_x}"
+      wheel_mount_point_x="${wheelbase/2.0}"
+      wheel_mount_point_y="${wheel_mount_point_y}"
       prefix="fr" />
     <xacro:wheel.wheel
       wheel_config="${wheel_config}"
-      wheel_separation_x="${wheel_separation_x}"
+      wheel_mount_point_x="${wheelbase/2.0}"
+      wheel_mount_point_y="${wheel_mount_point_y}"
       prefix="rl" />
     <xacro:wheel.wheel
       wheel_config="${wheel_config}"
-      wheel_separation_x="${wheel_separation_x}"
+      wheel_mount_point_x="${wheelbase/2.0}"
+      wheel_mount_point_y="${wheel_mount_point_y}"
       prefix="rr" />
     <ros2_control name="${ns}lynx_system" type="system">

File: husarion_ugv_description/urdf/panther/panther_macro.urdf.xacro (robot description, xacro)
@@ -16,5 +16,6 @@
     <xacro:property name="ns" value='${namespace + "/" if namespace else ""}' />
     <xacro:property name="wheel_config" value="${xacro.load_yaml(wheel_config_file)}" />
-    <xacro:property name="wheel_separation_x" value="0.44" />
+    <xacro:property name="wheelbase" value="0.44" />
+    <xacro:property name="wheel_mount_point_y" value="0.2575" />
     <!-- INCLUDE ROBOT PARTS DEFINITIONS -->
     <xacro:include filename="$(find husarion_ugv_description)/urdf/panther/base.urdf.xacro" ns="body" />
@@ -29,17 +30,21 @@
     <xacro:wheel.wheel
       wheel_config="${wheel_config}"
-      wheel_separation_x="${wheel_separation_x}"
+      wheel_mount_point_x="${wheelbase/2.0}"
+      wheel_mount_point_y="${wheel_mount_point_y}"
       prefix="fl" />
     <xacro:wheel.wheel
       wheel_config="${wheel_config}"
-      wheel_separation_x="${wheel_separation_x}"
+      wheel_mount_point_x="${wheelbase/2.0}"
+      wheel_mount_point_y="${wheel_mount_point_y}"
       prefix="fr" />
     <xacro:wheel.wheel
       wheel_config="${wheel_config}"
-      wheel_separation_x="${wheel_separation_x}"
+      wheel_mount_point_x="${wheelbase/2.0}"
+      wheel_mount_point_y="${wheel_mount_point_y}"
       prefix="rl" />
     <xacro:wheel.wheel
       wheel_config="${wheel_config}"
-      wheel_separation_x="${wheel_separation_x}"
+      wheel_mount_point_x="${wheelbase/2.0}"
+      wheel_mount_point_y="${wheel_mount_point_y}"
       prefix="rr" />
     <ros2_control name="${ns}panther_system" type="system">
