Commit message: review fixes

File: husarion_ugv_description/urdf/common/wheel.urdf.xacro (robot description, xacro)
@@ -2,37 +2,36 @@
 <robot xmlns:xacro="http://wiki.ros.org/xacro">
   <!-- wheel defining macro -->
-  <xacro:macro name="wheel"
-    params="wheel_config prefix wheel_mount_point_x wheel_mount_point_y">
+  <xacro:macro name="wheel" params="config prefix mount_point_x mount_point_y">
     <xacro:if value="${prefix == 'fl'}">
-      <xacro:property name="x" value="${wheel_mount_point_x}" />
-      <xacro:property name="y" value="${wheel_mount_point_y}" />
-      <xacro:property name="mount_point_offset" value="${wheel_config['mount_point_offset']}" />
-      <xacro:property name="inertia_y_offset" value="${wheel_config['inertia_y_offset']}" />
+      <xacro:property name="x" value="${mount_point_x}" />
+      <xacro:property name="y" value="${mount_point_y}" />
+      <xacro:property name="mount_point_offset" value="${config['mount_point_offset']}" />
+      <xacro:property name="inertia_y_offset" value="${config['inertia_y_offset']}" />
       <xacro:property name="fdir" value="1 -1 0" />
     </xacro:if>
     <xacro:if value="${prefix == 'fr'}">
-      <xacro:property name="x" value="${wheel_mount_point_x}" />
-      <xacro:property name="y" value="-${wheel_mount_point_y}" />
-      <xacro:property name="mount_point_offset" value="-${wheel_config['mount_point_offset']}" />
-      <xacro:property name="inertia_y_offset" value="${-wheel_config['inertia_y_offset']}" />
+      <xacro:property name="x" value="${mount_point_x}" />
+      <xacro:property name="y" value="-${mount_point_y}" />
+      <xacro:property name="mount_point_offset" value="-${config['mount_point_offset']}" />
+      <xacro:property name="inertia_y_offset" value="${-config['inertia_y_offset']}" />
       <xacro:property name="fdir" value="1 1 0" />
     </xacro:if>
     <xacro:if value="${prefix == 'rl'}">
-      <xacro:property name="x" value="-${wheel_mount_point_x}" />
-      <xacro:property name="y" value="${wheel_mount_point_y}" />
-      <xacro:property name="mount_point_offset" value="${wheel_config['mount_point_offset']}" />
-      <xacro:property name="inertia_y_offset" value="${wheel_config['inertia_y_offset']}" />
+      <xacro:property name="x" value="-${mount_point_x}" />
+      <xacro:property name="y" value="${mount_point_y}" />
+      <xacro:property name="mount_point_offset" value="${config['mount_point_offset']}" />
+      <xacro:property name="inertia_y_offset" value="${config['inertia_y_offset']}" />
       <xacro:property name="fdir" value="1 1 0" />
     </xacro:if>
     <xacro:if value="${prefix == 'rr'}">
-      <xacro:property name="x" value="-${wheel_mount_point_x}" />
-      <xacro:property name="y" value="-${wheel_mount_point_y}" />
-      <xacro:property name="mount_point_offset" value="-${wheel_config['mount_point_offset']}" />
-      <xacro:property name="inertia_y_offset" value="${-wheel_config['inertia_y_offset']}" />
+      <xacro:property name="x" value="-${mount_point_x}" />
+      <xacro:property name="y" value="-${mount_point_y}" />
+      <xacro:property name="mount_point_offset" value="-${config['mount_point_offset']}" />
+      <xacro:property name="inertia_y_offset" value="${-config['inertia_y_offset']}" />
       <xacro:property name="fdir" value="1 -1 0" />
     </xacro:if>
-    <joint name="base_to_${prefix}_wheel_base_joint" type="fixed">
+    <joint name="body_to_${prefix}_wheel_base_joint" type="fixed">
       <origin xyz="${x} ${y} 0.0" rpy="0.0 0.0 0.0" />
-      <parent link="base_link" />
+      <parent link="body_link" />
       <child link="${prefix}_wheel_base_link" />
     </joint>
@@ -50,5 +49,5 @@
         <origin xyz="0.0 0.0 0.0" rpy="0.0 0.0 0.0" />
         <geometry>
-          <mesh filename="package://${wheel_config['mesh_package']}/${wheel_config['folder_path']}/${prefix}_wheel.dae" />
+          <mesh filename="package://${config['mesh_package']}/${config['folder_path']}/${prefix}_wheel.dae" />
         </geometry>
       </visual>
@@ -56,21 +55,21 @@
         <origin xyz="0.0 0.0 0.0" rpy="-${pi/2} 0.0 0.0" />
         <geometry>
-          <cylinder radius="${wheel_config['wheel_radius']}" length="${wheel_config['wheel_width']}" />
+          <cylinder radius="${config['wheel_radius']}" length="${config['wheel_width']}" />
         </geometry>
       </collision>
       <inertial>
         <origin xyz="0.0 ${inertia_y_offset} 0.0" rpy="0.0 0.0 0.0" />
-        <mass value="${wheel_config['mass']}" />
+        <mass value="${config['mass']}" />
         <inertia
-          ixx="${wheel_config['inertia']['ixx']}"
+          ixx="${config['inertia']['ixx']}"
           ixy="0.0"
           ixz="0.0"
-          iyy="${wheel_config['inertia']['iyy']}"
+          iyy="${config['inertia']['iyy']}"
           iyz="0.0"
-          izz="${wheel_config['inertia']['izz']}" />
+          izz="${config['inertia']['izz']}" />
       </inertial>
     </link>
     <xacro:if value="${use_sim}">
-      <xacro:if value="${wheel_config['mecanum']}">
+      <xacro:if value="${config['mecanum']}">
         <gazebo reference="${prefix}_wheel_link" xmlns:ignition="http://ignitionrobotics.org/schema">
           <collision>

File: husarion_ugv_description/urdf/lynx/base.urdf.xacro (robot description, xacro)
@@ -4,5 +4,11 @@
     name="body"
     params="wheel_radius imu_xyz imu_rpy">
-    <link name="base_link">
+    <joint name="base_to_body_joint" type="fixed">
+      <origin xyz="0.0 0.0 0.0" rpy="0.0 0.0 0.0" />
+      <parent link="base_link" />
+      <child link="body_link" />
+    </joint>
+    <link name="base_link" />
+    <link name="body_link">
       <visual>
         <geometry>
@@ -24,19 +30,19 @@
       </inertial>
     </link>
-    <joint name="base_to_footprint_joint" type="fixed">
+    <joint name="body_to_footprint_joint" type="fixed">
       <origin xyz="0.0 0.0 -${wheel_radius}" rpy="0.0 0.0 0.0" />
-      <parent link="base_link" />
+      <parent link="body_link" />
       <child link="base_footprint" />
     </joint>
     <link name="base_footprint" />
-    <joint name="base_to_imu_joint" type="fixed">
+    <joint name="body_to_imu_joint" type="fixed">
       <origin xyz="${imu_xyz}" rpy="${imu_rpy}" />
-      <parent link="base_link" />
+      <parent link="body_link" />
       <child link="imu_link" />
     </joint>
     <link name="imu_link" />
-    <joint name="base_to_cover_joint" type="fixed">
+    <joint name="body_to_cover_joint" type="fixed">
       <origin xyz="0.0 0.0 0.2098" rpy="0.0 0.0 0.0" />
-      <parent link="base_link" />
+      <parent link="body_link" />
       <child link="cover_link" />
     </joint>

File: husarion_ugv_description/urdf/lynx/lynx_macro.urdf.xacro (robot description, xacro)
@@ -25,22 +25,22 @@
     <!-- WHEEL DECLARATION -->
     <xacro:wheel.wheel
-      wheel_config="${wheel_config}"
-      wheel_mount_point_x="${wheelbase/2.0}"
-      wheel_mount_point_y="${wheel_mount_point_y}"
+      config="${wheel_config}"
+      mount_point_x="${wheelbase/2.0}"
+      mount_point_y="${wheel_mount_point_y}"
       prefix="fl" />
     <xacro:wheel.wheel
-      wheel_config="${wheel_config}"
-      wheel_mount_point_x="${wheelbase/2.0}"
-      wheel_mount_point_y="${wheel_mount_point_y}"
+      config="${wheel_config}"
+      mount_point_x="${wheelbase/2.0}"
+      mount_point_y="${wheel_mount_point_y}"
       prefix="fr" />
     <xacro:wheel.wheel
-      wheel_config="${wheel_config}"
-      wheel_mount_point_x="${wheelbase/2.0}"
-      wheel_mount_point_y="${wheel_mount_point_y}"
+      config="${wheel_config}"
+      mount_point_x="${wheelbase/2.0}"
+      mount_point_y="${wheel_mount_point_y}"
       prefix="rl" />
     <xacro:wheel.wheel
-      wheel_config="${wheel_config}"
-      wheel_mount_point_x="${wheelbase/2.0}"
-      wheel_mount_point_y="${wheel_mount_point_y}"
+      config="${wheel_config}"
+      mount_point_x="${wheelbase/2.0}"
+      mount_point_y="${wheel_mount_point_y}"
       prefix="rr" />
     <ros2_control name="${ns}lynx_system" type="system">

File: husarion_ugv_description/urdf/panther/base.urdf.xacro (robot description, xacro)
@@ -1,11 +1,15 @@
 <?xml version="1.0" encoding="utf-8"?>
 <robot xmlns:xacro="http://wiki.ros.org/xacro">
-  <!-- body defining macro -->
   <xacro:macro
     name="body"
     params="wheel_radius imu_xyz imu_rpy">
-    <link name="base_link">
+    <joint name="base_to_body_joint" type="fixed">
+      <origin xyz="0.0 0.0 0.0" rpy="0.0 0.0 0.0" />
+      <parent link="base_link" />
+      <child link="body_link" />
+    </joint>
+    <link name="base_link" />
+    <link name="body_link">
       <visual>
-        <origin xyz="0.0 0.0 0.0" rpy="0.0 0.0 0.0" />
         <geometry>
           <mesh filename="package://husarion_ugv_description/meshes/panther/base.dae" />
@@ -26,19 +30,19 @@
       </inertial>
     </link>
-    <joint name="base_to_footprint_joint" type="fixed">
+    <joint name="body_to_footprint_joint" type="fixed">
       <origin xyz="0.0 0.0 -${wheel_radius}" rpy="0.0 0.0 0.0" />
-      <parent link="base_link" />
+      <parent link="body_link" />
       <child link="base_footprint" />
     </joint>
     <link name="base_footprint" />
-    <joint name="base_to_imu_joint" type="fixed">
+    <joint name="body_to_imu_joint" type="fixed">
       <origin xyz="${imu_xyz}" rpy="${imu_rpy}" />
-      <parent link="base_link" />
+      <parent link="body_link" />
       <child link="imu_link" />
     </joint>
     <link name="imu_link" />
-    <joint name="base_to_front_bumper_joint" type="fixed">
+    <joint name="body_to_front_bumper_joint" type="fixed">
       <origin xyz="0.362 0.0 0.0" rpy="0.0 0.0 0.0" />
-      <parent link="base_link" />
+      <parent link="body_link" />
       <child link="front_bumper_link" />
     </joint>
@@ -50,7 +54,7 @@
     </joint>
     <link name="lights_channel_1_link" />
-    <joint name="base_to_rear_bumper_joint" type="fixed">
+    <joint name="body_to_rear_bumper_joint" type="fixed">
       <origin xyz="-0.362 0.0 0.0" rpy="0.0 0.0 ${pi}" />
-      <parent link="base_link" />
+      <parent link="body_link" />
       <child link="rear_bumper_link" />
     </joint>
@@ -62,7 +66,7 @@
     </joint>
     <link name="lights_channel_2_link" />
-    <joint name="base_to_cover_joint" type="fixed">
+    <joint name="body_to_cover_joint" type="fixed">
       <origin xyz="0.0 0.0 0.14" rpy="0.0 0.0 0.0" />
-      <parent link="base_link" />
+      <parent link="body_link" />
       <child link="cover_link" />
     </joint>

File: husarion_ugv_description/urdf/panther/panther_macro.urdf.xacro (robot description, xacro)
@@ -29,22 +29,22 @@
     <!-- WHEEL DECLARATION -->
     <xacro:wheel.wheel
-      wheel_config="${wheel_config}"
-      wheel_mount_point_x="${wheelbase/2.0}"
-      wheel_mount_point_y="${wheel_mount_point_y}"
+      config="${wheel_config}"
+      mount_point_x="${wheelbase/2.0}"
+      mount_point_y="${wheel_mount_point_y}"
       prefix="fl" />
     <xacro:wheel.wheel
-      wheel_config="${wheel_config}"
-      wheel_mount_point_x="${wheelbase/2.0}"
-      wheel_mount_point_y="${wheel_mount_point_y}"
+      config="${wheel_config}"
+      mount_point_x="${wheelbase/2.0}"
+      mount_point_y="${wheel_mount_point_y}"
       prefix="fr" />
     <xacro:wheel.wheel
-      wheel_config="${wheel_config}"
-      wheel_mount_point_x="${wheelbase/2.0}"
-      wheel_mount_point_y="${wheel_mount_point_y}"
+      config="${wheel_config}"
+      mount_point_x="${wheelbase/2.0}"
+      mount_point_y="${wheel_mount_point_y}"
       prefix="rl" />
     <xacro:wheel.wheel
-      wheel_config="${wheel_config}"
-      wheel_mount_point_x="${wheelbase/2.0}"
-      wheel_mount_point_y="${wheel_mount_point_y}"
+      config="${wheel_config}"
+      mount_point_x="${wheelbase/2.0}"
+      mount_point_y="${wheel_mount_point_y}"
       prefix="rr" />
     <ros2_control name="${ns}panther_system" type="system">
