Commit message: Update husarion_ugv_description/urdf/common/gazebo.urdf.xacro

File: husarion_ugv_description/urdf/common/gazebo.urdf.xacro (robot description, xacro)
@@ -60,5 +60,5 @@
   <!-- IMU specification: https://www.phidgets.com/?tier=3&catid=10&pcid=8&prodid=1025#Tab_Specifications -->
   <xacro:macro name="imu" params="reference_frame namespace:=''">
-  <xacro:property name="ns" value='${namespace + "/" if namespace else ""}' />
+    <xacro:property name="ns" value='${namespace + "/" if namespace else ""}' />
     <gazebo reference="${reference_frame}">
       <sensor name="${ns}imu" type="imu">

Commit message: add ground truth odometry and tf

File: husarion_ugv_description/urdf/common/gazebo.urdf.xacro (robot description, xacro)
@@ -133,3 +133,18 @@
     </gazebo>
   </xacro:macro>
+  <xacro:macro name="odometry_publisher" params="namespace:=''">
+    <xacro:property name="ns" value='${namespace + "/" if namespace else ""}' />
+    <gazebo>
+      <plugin
+        filename="gz-sim-odometry-publisher-system"
+        name="gz::sim::systems::OdometryPublisher">
+        <odom_frame>world</odom_frame>
+        <robot_base_frame>${ns}base_link</robot_base_frame>
+        <odom_topic>${ns}odometry/ground_truth</odom_topic>
+        <odom_covariance_topic>${ns}odometry/ground_truth_covariance</odom_covariance_topic>
+        <tf_topic>tf_gt</tf_topic>
+        <odom_publish_frequency>50.0</odom_publish_frequency>
+      </plugin>
+    </gazebo>
+  </xacro:macro>
 </robot>

File: husarion_ugv_description/urdf/panther/panther_macro.urdf.xacro (robot description, xacro)
@@ -163,4 +163,5 @@
       <xacro:gazebo.light reference_frame="lights_channel_1_link" name="lights_channel_1" topic="lights/channel_1_frame" namespace="${namespace}" />
       <xacro:gazebo.light reference_frame="lights_channel_2_link" name="lights_channel_2" topic="lights/channel_2_frame" namespace="${namespace}" />
+      <xacro:gazebo.odometry_publisher namespace="${namespace}" />
     </xacro:if>
   </xacro:macro>

Commit message: Rework simulation e-stop and LED strip visualization
Standalone e-stop plugin actually stops the robot and fixes #623;
LED strips follow a polyline (4 Lynx corner segments) and markers
are re-sent only when LED colors change.

File: husarion_ugv_description/urdf/common/gazebo.urdf.xacro (robot description, xacro)
@@ -43,4 +43,15 @@
           <remapping>twist_mux_controller/transition_event:=twist_mux_controller/_transition_event</remapping>
         </ros>
+      </plugin>
+    </gazebo>
+  </xacro:macro>
+  <!-- E-stop -->
+  <!-- Must be declared after the controller macro: gz-sim executes systems in declaration order
+       and the E-stop zeros have to overwrite the commands written by gz_ros2_control. -->
+  <xacro:macro name="estop" params="namespace:='' initial_state:=true">
+    <gazebo>
+      <plugin filename="EStopSystem" name="husarion_ugv_gazebo::EStopSystem">
+        <namespace>${namespace}</namespace>
+        <initial_state>${initial_state}</initial_state>
       </plugin>
     </gazebo>
@@ -101,5 +112,8 @@
   </xacro:macro>
   <!-- Lights -->
-  <xacro:macro name="light" params="reference_frame name topic namespace:=''">
+  <!-- led_range selects a "first-last" subrange of the channel frame (reversed range flips the
+       LED order); points defines a polyline ("x y z; x y z; ...", in the light frame) the LEDs
+       are placed along. With no points the strip is a straight line of the given width. -->
+  <xacro:macro name="light" params="reference_frame name topic namespace:='' led_range:='' points:='' width:=0.5 height:=0.015 light_type:=spot light_direction:='1 0 0' spot_inner_angle:=1.0 spot_outer_angle:=2.0">
     <gazebo>
       <plugin filename="LEDStrip" name="husarion_ugv_gazebo::LEDStrip">
@@ -108,21 +122,29 @@
         <namespace>${namespace}</namespace>
         <frequency>10</frequency>
-        <width>0.5</width>
-        <height>0.015</height>
+        <width>${width}</width>
+        <height>${height}</height>
+        <xacro:if value="${led_range != ''}">
+          <led_range>${led_range}</led_range>
+        </xacro:if>
+        <xacro:if value="${points != ''}">
+          <points>${points}</points>
+        </xacro:if>
       </plugin>
     </gazebo>
     <gazebo reference="${reference_frame}">
-      <light name="${name}" type="spot">
+      <light name="${name}" type="${light_type}">
         <cast_shadows>true</cast_shadows>
         <visualize>0</visualize>
         <diffuse>1.0 1.0 1.0</diffuse>
         <specular>1.0 1.0 1.0</specular>
-        <direction>1 0 0</direction>
         <intensity>0.5</intensity>
-        <spot>
-          <inner_angle>1.0</inner_angle>
-          <outer_angle>2.0</outer_angle>
-          <falloff>0.4</falloff>
-        </spot>
+        <xacro:if value="${light_type == 'spot'}">
+          <direction>${light_direction}</direction>
+          <spot>
+            <inner_angle>${spot_inner_angle}</inner_angle>
+            <outer_angle>${spot_outer_angle}</outer_angle>
+            <falloff>0.4</falloff>
+          </spot>
+        </xacro:if>
         <attenuation>
           <range>20.0</range>

File: husarion_ugv_description/urdf/lynx/lynx_macro.urdf.xacro (robot description, xacro)
@@ -52,6 +52,5 @@
       <hardware>
         <xacro:if value="${use_sim}">
-          <plugin>husarion_ugv_gazebo/EStopSystem</plugin>
-          <param name="e_stop_initial_state">true</param>
+          <plugin>gz_ros2_control/GazeboSimSystem</plugin>
         </xacro:if>
         <xacro:unless value="${use_sim}">
@@ -161,8 +160,16 @@
       </xacro:if>
       <xacro:gazebo.controller config_file="${controller_config_file}" namespace="${namespace}" />
+      <xacro:gazebo.estop namespace="${namespace}" />
       <xacro:gazebo.imu reference_frame="imu_link" namespace="${namespace}" />
-      <!-- TODO Add lights visualization -->
-      <!-- <xacro:gazebo.light reference_frame="lights_channel_1_link" name="lights_channel_1" topic="lights/channel_1_frame" namespace="${namespace}" /> -->
-      <!-- <xacro:gazebo.light reference_frame="lights_channel_2_link" name="lights_channel_2" topic="lights/channel_2_frame" namespace="${namespace}" /> -->
+      <!-- Corner LED strips. Front: a straight 5 cm strip angled 60 deg to the front fascia,
+           rising from 0.15 m (inner end) to 0.18 m (outer end). Rear: a U-shaped strip (inner
+           edge, back, outer edge). Channel layout from lynx_animations.yaml: channel 1 fl=23-12
+           rl=0-11, channel 2 fr=23-12 rr=0-11. -->
+      <!-- Wide downward-facing spots approximate a strip glowing radially in the horizontal
+           plane (no light cast into the sky). -->
+      <xacro:gazebo.light reference_frame="lights_fl_link" name="lights_fl" topic="lights/channel_1_frame" namespace="${namespace}" spot_outer_angle="1.5" led_range="23-12" points="-0.01 -0.065 0.0; 0.0 -0.063 0.0; 0.005 0.056 0.0" />
+      <xacro:gazebo.light reference_frame="lights_fr_link" name="lights_fr" topic="lights/channel_2_frame" namespace="${namespace}" spot_outer_angle="1.5" led_range="23-12" points="-0.01 0.065 0.0; 0.0 0.063 0.0; 0.005 -0.056 0.0" />
+      <xacro:gazebo.light reference_frame="lights_rl_link" name="lights_rl" topic="lights/channel_1_frame" namespace="${namespace}" spot_outer_angle="3.0" led_range="0-11" points="-0.029 0.04 0.01; 0.0 0.023 0.006; 0.006 -0.03 -0.005; -0.067 -0.035 -0.005" />
+      <xacro:gazebo.light reference_frame="lights_rr_link" name="lights_rr" topic="lights/channel_2_frame" namespace="${namespace}" spot_outer_angle="3.0" led_range="0-11" points="-0.029 -0.04 0.01; 0.0 -0.023 0.006; 0.006 0.03 -0.005; -0.067 0.035 -0.005" />
       <xacro:gazebo.odometry_publisher namespace="${namespace}" />
     </xacro:if>

File: husarion_ugv_description/urdf/panther/panther_macro.urdf.xacro (robot description, xacro)
@@ -52,6 +52,5 @@
       <hardware>
         <xacro:if value="${use_sim}">
-          <plugin>husarion_ugv_gazebo/EStopSystem</plugin>
-          <param name="e_stop_initial_state">true</param>
+          <plugin>gz_ros2_control/GazeboSimSystem</plugin>
         </xacro:if>
         <xacro:unless value="${use_sim}">
@@ -162,4 +161,5 @@
       </xacro:if>
       <xacro:gazebo.controller config_file="${controller_config_file}" namespace="${namespace}" />
+      <xacro:gazebo.estop namespace="${namespace}" />
       <xacro:gazebo.imu reference_frame="imu_link" namespace="${namespace}" />
       <xacro:gazebo.light reference_frame="lights_channel_1_link" name="lights_channel_1" topic="lights/channel_1_frame" namespace="${namespace}" />

Commit message: Add LED diffuser blur, lights launch toggle, gz logging macros
Replace deprecated ign* logging macros with gz*; add a 'lights' launch
arg to disable the simulated LED controller; add an optional 1D Gaussian
blur (blur_sigma) approximating the LED diffuser.

File: husarion_ugv_description/urdf/common/gazebo.urdf.xacro (robot description, xacro)
@@ -115,5 +115,5 @@
        LED order); points defines a polyline ("x y z; x y z; ...", in the light frame) the LEDs
        are placed along. With no points the strip is a straight line of the given width. -->
-  <xacro:macro name="light" params="reference_frame name topic namespace:='' led_range:='' points:='' width:=0.5 height:=0.015 light_type:=spot light_direction:='1 0 0' spot_inner_angle:=1.0 spot_outer_angle:=2.0">
+  <xacro:macro name="light" params="reference_frame name topic namespace:='' led_range:='' points:='' width:=0.5 height:=0.015 light_type:=spot light_direction:='1 0 0' spot_inner_angle:=1.0 spot_outer_angle:=2.0 blur_sigma:=0.8">
     <gazebo>
       <plugin filename="LEDStrip" name="husarion_ugv_gazebo::LEDStrip">
@@ -124,4 +124,5 @@
         <width>${width}</width>
         <height>${height}</height>
+        <blur_sigma>${blur_sigma}</blur_sigma>
         <xacro:if value="${led_range != ''}">
           <led_range>${led_range}</led_range>

File: husarion_ugv_description/urdf/lynx/lynx_macro.urdf.xacro (robot description, xacro)
@@ -168,8 +168,8 @@
       <!-- Wide downward-facing spots approximate a strip glowing radially in the horizontal
            plane (no light cast into the sky). -->
-      <xacro:gazebo.light reference_frame="lights_fl_link" name="lights_fl" topic="lights/channel_1_frame" namespace="${namespace}" spot_outer_angle="1.5" led_range="23-12" points="-0.01 -0.065 0.0; 0.0 -0.063 0.0; 0.005 0.056 0.0" />
-      <xacro:gazebo.light reference_frame="lights_fr_link" name="lights_fr" topic="lights/channel_2_frame" namespace="${namespace}" spot_outer_angle="1.5" led_range="23-12" points="-0.01 0.065 0.0; 0.0 0.063 0.0; 0.005 -0.056 0.0" />
-      <xacro:gazebo.light reference_frame="lights_rl_link" name="lights_rl" topic="lights/channel_1_frame" namespace="${namespace}" spot_outer_angle="3.0" led_range="0-11" points="-0.029 0.04 0.01; 0.0 0.023 0.006; 0.006 -0.03 -0.005; -0.067 -0.035 -0.005" />
-      <xacro:gazebo.light reference_frame="lights_rr_link" name="lights_rr" topic="lights/channel_2_frame" namespace="${namespace}" spot_outer_angle="3.0" led_range="0-11" points="-0.029 -0.04 0.01; 0.0 -0.023 0.006; 0.006 0.03 -0.005; -0.067 0.035 -0.005" />
+      <xacro:gazebo.light reference_frame="lights_fl_link" name="lights_fl" topic="lights/channel_1_frame" namespace="${namespace}" spot_outer_angle="1.5" led_range="23-12" points="-0.01 -0.065 0.0; 0.0 -0.058 0.0; 0.005 0.056 0.0" />
+      <xacro:gazebo.light reference_frame="lights_fr_link" name="lights_fr" topic="lights/channel_2_frame" namespace="${namespace}" spot_outer_angle="1.5" led_range="23-12" points="-0.01 0.065 0.0; 0.0 0.058 0.0; 0.005 -0.056 0.0" />
+      <xacro:gazebo.light reference_frame="lights_rl_link" name="lights_rl" topic="lights/channel_1_frame" namespace="${namespace}" spot_outer_angle="3.0" led_range="0-11" points="-0.027 0.04 0.01; -0.002 0.025 0.007; 0.006 -0.018 -0.002; -0.002 -0.03 -0.005; -0.067 -0.035 -0.005" />
+      <xacro:gazebo.light reference_frame="lights_rr_link" name="lights_rr" topic="lights/channel_2_frame" namespace="${namespace}" spot_outer_angle="3.0" led_range="0-11" points="-0.027 -0.04 0.01; -0.002 -0.025 0.007; 0.006 0.018 -0.002; -0.002 0.03 -0.005; -0.067 0.035 -0.005" />
       <xacro:gazebo.odometry_publisher namespace="${namespace}" />
     </xacro:if>

Commit message: Fix LED strip sim slowdown, drop lights launch toggle
VisualizeLights appended to the persistent light_cmd_ header every frame; the message grew unboundedly and dragged the real-time factor down over time.

File: husarion_ugv_description/urdf/common/gazebo.urdf.xacro (robot description, xacro)
@@ -115,5 +115,5 @@
        LED order); points defines a polyline ("x y z; x y z; ...", in the light frame) the LEDs
        are placed along. With no points the strip is a straight line of the given width. -->
-  <xacro:macro name="light" params="reference_frame name topic namespace:='' led_range:='' points:='' width:=0.5 height:=0.015 light_type:=spot light_direction:='1 0 0' spot_inner_angle:=1.0 spot_outer_angle:=2.0 blur_sigma:=0.8">
+  <xacro:macro name="light" params="reference_frame name topic namespace:='' led_range:='' points:='' width:=0.5 height:=0.015 light_type:=spot light_direction:='1 0 0' spot_inner_angle:=1.0 spot_outer_angle:=2.0 blur_sigma:=1.3">
     <gazebo>
       <plugin filename="LEDStrip" name="husarion_ugv_gazebo::LEDStrip">

File: husarion_ugv_description/urdf/lynx/lynx_macro.urdf.xacro (robot description, xacro)
@@ -168,6 +168,6 @@
       <!-- Wide downward-facing spots approximate a strip glowing radially in the horizontal
            plane (no light cast into the sky). -->
-      <xacro:gazebo.light reference_frame="lights_fl_link" name="lights_fl" topic="lights/channel_1_frame" namespace="${namespace}" spot_outer_angle="1.5" led_range="23-12" points="-0.01 -0.065 0.0; 0.0 -0.058 0.0; 0.005 0.056 0.0" />
-      <xacro:gazebo.light reference_frame="lights_fr_link" name="lights_fr" topic="lights/channel_2_frame" namespace="${namespace}" spot_outer_angle="1.5" led_range="23-12" points="-0.01 0.065 0.0; 0.0 0.058 0.0; 0.005 -0.056 0.0" />
+      <xacro:gazebo.light reference_frame="lights_fl_link" name="lights_fl" topic="lights/channel_1_frame" namespace="${namespace}" spot_outer_angle="1.5" led_range="23-12" points="-0.01 -0.066 0.0; 0.0 -0.058 0.0; 0.003 0.056 0.0" />
+      <xacro:gazebo.light reference_frame="lights_fr_link" name="lights_fr" topic="lights/channel_2_frame" namespace="${namespace}" spot_outer_angle="1.5" led_range="23-12" points="-0.01 0.066 0.0; 0.0 0.058 0.0; 0.003 -0.056 0.0" />
       <xacro:gazebo.light reference_frame="lights_rl_link" name="lights_rl" topic="lights/channel_1_frame" namespace="${namespace}" spot_outer_angle="3.0" led_range="0-11" points="-0.027 0.04 0.01; -0.002 0.025 0.007; 0.006 -0.018 -0.002; -0.002 -0.03 -0.005; -0.067 -0.035 -0.005" />
       <xacro:gazebo.light reference_frame="lights_rr_link" name="lights_rr" topic="lights/channel_2_frame" namespace="${namespace}" spot_outer_angle="3.0" led_range="0-11" points="-0.027 -0.04 0.01; -0.002 -0.025 0.007; 0.006 0.018 -0.002; -0.002 0.03 -0.005; -0.067 0.035 -0.005" />

Commit message: Rework sim LED diffuser: gradient, white base, marker batch
Gaussian blur width scaled with LED resolution and bled across gaps (MANUAL_ACTION's two bars merged); replace with a local sub-LED gradient. Composite over a white base so transparent animations reveal the diffuser instead of going black. Run-merge equal-color cells + one batched /marker_array request fix the full-strip-fade GUI stutter.

File: husarion_ugv_description/urdf/common/gazebo.urdf.xacro (robot description, xacro)
@@ -115,5 +115,5 @@
        LED order); points defines a polyline ("x y z; x y z; ...", in the light frame) the LEDs
        are placed along. With no points the strip is a straight line of the given width. -->
-  <xacro:macro name="light" params="reference_frame name topic namespace:='' led_range:='' points:='' width:=0.5 height:=0.015 light_type:=spot light_direction:='1 0 0' spot_inner_angle:=1.0 spot_outer_angle:=2.0 blur_sigma:=1.3">
+  <xacro:macro name="light" params="reference_frame name topic namespace:='' led_range:='' points:='' width:=0.5 height:=0.015 light_type:=spot light_direction:='1 0 0' spot_inner_angle:=1.0 spot_outer_angle:=2.0 render_markers_per_led:=1 strip_base_color:='1 1 1'">
     <gazebo>
       <plugin filename="LEDStrip" name="husarion_ugv_gazebo::LEDStrip">
@@ -124,5 +124,6 @@
         <width>${width}</width>
         <height>${height}</height>
-        <blur_sigma>${blur_sigma}</blur_sigma>
+        <render_markers_per_led>${render_markers_per_led}</render_markers_per_led>
+        <strip_base_color>${strip_base_color}</strip_base_color>
         <xacro:if value="${led_range != ''}">
           <led_range>${led_range}</led_range>

Commit message: Dawid suggestions

File: husarion_ugv_description/urdf/common/gazebo.urdf.xacro (robot description, xacro)
@@ -115,5 +115,5 @@
        LED order); points defines a polyline ("x y z; x y z; ...", in the light frame) the LEDs
        are placed along. With no points the strip is a straight line of the given width. -->
-  <xacro:macro name="light" params="reference_frame name topic namespace:='' led_range:='' points:='' width:=0.5 height:=0.015 light_type:=spot light_direction:='1 0 0' spot_inner_angle:=1.0 spot_outer_angle:=2.0 render_markers_per_led:=1 strip_base_color:='1 1 1'">
+  <xacro:macro name="light" params="reference_frame name topic namespace:='' led_range:='' points:='' width:=0.5 height:=0.015 light_type:=spot light_direction:='1 0 0' spot_inner_angle:=1.0 spot_outer_angle:=2.0 render_markers_per_led:=2 strip_base_color:='1 1 1'">
     <gazebo>
       <plugin filename="LEDStrip" name="husarion_ugv_gazebo::LEDStrip">

Commit message: Additive LED diffuser wash so dim colors keep hue

File: husarion_ugv_description/urdf/common/gazebo.urdf.xacro (robot description, xacro)
@@ -115,5 +115,5 @@
        LED order); points defines a polyline ("x y z; x y z; ...", in the light frame) the LEDs
        are placed along. With no points the strip is a straight line of the given width. -->
-  <xacro:macro name="light" params="reference_frame name topic namespace:='' led_range:='' points:='' width:=0.5 height:=0.015 light_type:=spot light_direction:='1 0 0' spot_inner_angle:=1.0 spot_outer_angle:=2.0 render_markers_per_led:=2 strip_base_color:='1 1 1'">
+  <xacro:macro name="light" params="reference_frame name topic namespace:='' led_range:='' points:='' width:=0.5 height:=0.015 light_type:=spot light_direction:='1 0 0' spot_inner_angle:=1.0 spot_outer_angle:=2.0 render_markers_per_led:=2 strip_base_color:='1 1 1 0.3'">
     <gazebo>
       <plugin filename="LEDStrip" name="husarion_ugv_gazebo::LEDStrip">
